File: Alpengluehn2.kicad_pcb (KiCad board)
At the start: 2 copper layers, 100 x 80 mm, 126 parts, among them IC2 PCA9685, P1 CONN_7X2, P2 CONN_5X2, P3 CONN_5X2, SW1 DIPS_06, U10 PT4115-SOT89-5, U11 PT4115-SOT89-5, U12 PT4115-SOT89-5, U13 PT4115-SOT89-5, U14 PT4115-SOT89-5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

Commit message: corrected drawing of power connector
Signed-off-by: Maximilian Güntner <maximilian.guentner@gmail.com>
Other:
- board text added: "GND"
